File: MCU Datalogger.kicad_sch (KiCad schematic)
At the start: 25 parts, among them U1 24LC1025, U2 24LC1025, U3 DS1337S_, U4 ATMEGA328P-AU, Y1 16MHz, Y2 32.768 KHz

Commit message: Final 2-layered PCB with Logo
Connections:
- net VCC: now also BT1.1 (+), C5.1, D2.2 (A), U4.18 (AVCC), U4.4 (VCC)
Changed lines of the file:
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@@
+		)
+	)
+	(label "VCC"
+		(at 265.43 35.56 0)
+		(effects
+			(font
+				(size 1.27 1.27)
+			)
+			(justify left bottom)
 		)
 	)

Commit message: Fixed two defects in the schematics
Connections:
- net SCK: no longer R1.2, U1.6 (SCL), U2.6 (SCL), U3.6 (SCL), U4.28 (PC5)
- new net SCL: R1.2, U1.6 (SCL), U2.6 (SCL), U3.6 (SCL), U4.28 (PC5)
Other:
- sheet Connectors Sheet ports: added SCL; removed none
Changed lines of the file:
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@@
 	(wire
 		(pts
-			(xy 257.81 29.21) (xy 257.81 35.56)
-		)
-		(stroke
-			(width 0)
-			(type default)
-		)
-	)
-	(wire
-		(pts
 			(xy 83.82 139.7) (xy 83.82 144.78)
 		)
@@
 		)
 	)
+	(label "SCL"
+		(at 151.13 135.89 180)
+		(effects
+			(font
+				(size 1.27 1.27)
+			)
+			(justify right bottom)
+		)
+	)
 	(label "D3"
 		(at 238.76 50.8 0)
@@
 		)
 	)
-	(label "SCK"
+	(label "SCL"
 		(at 208.28 78.74 180)
 		(effects
@@
 		)
 	)
+	(label "SCL"
+		(at 83.82 137.16 0)
+		(effects
+			(font
+				(size 1.27 1.27)
+			)
+			(justify left bottom)
+		)
+	)
 	(label "VCC"
 		(at 63.5 134.62 180)
@@
 		)
 	)
-	(label "SCK"
+	(label "SCL"
 		(at 35.56 34.29 180)
 		(effects
@@
 		)
 	)
-	(label "SCK"
-		(at 45.72 137.16 0)
-		(effects
-			(font
-				(size 1.27 1.27)
-			)
-			(justify left bottom)
-		)
-	)
-	(label "SCK"
-		(at 95.25 144.78 180)
-		(effects
-			(font
-				(size 1.27 1.27)
-			)
-			(justify right bottom)
-		)
-	)
 	(label "D4"
 		(at 185.42 133.35 0)
@@
 	)
 	(label "RESET"
-		(at 151.13 151.13 180)
+		(at 151.13 152.4 180)
+		(effects
+			(font
+				(size 1.27 1.27)
+			)
+			(justify right bottom)
+		)
+	)
+	(label "SCK"
+		(at 151.13 138.43 180)
 		(effects
 			(font
@@
 	)
 	(label "SDA"
-		(at 151.13 132.08 180)
+		(at 151.13 133.35 180)
+		(effects
+			(font
+				(size 1.27 1.27)
+			)
+			(justify right bottom)
+		)
+	)
+	(label "SCL"
+		(at 95.25 144.78 180)
 		(effects
 			(font
@@
 	)
 	(label "MISO"
-		(at 151.13 139.7 180)
+		(at 151.13 146.05 180)
 		(effects
 			(font
@@
 		)
 	)
-	(label "SCK"
-		(at 83.82 137.16 0)
-		(effects
-			(font
-				(size 1.27 1.27)
-			)
-			(justify left bottom)
-		)
-	)
 	(label "MOSI"
-		(at 151.13 143.51 180)
+		(at 151.13 148.59 180)
 		(effects
 			(font
@@
 		)
 	)
-	(label "SCK"
-		(at 208.28 55.88 180)
+	(label "SCL"
+		(at 45.72 137.16 0)
 		(effects
 			(font
 				(size 1.27 1.27)
 			)
-			(justify right bottom)
+			(justify left bottom)
 		)
 	)
 	(label "SCK"
-		(at 151.13 134.62 180)
+		(at 208.28 55.88 180)
 		(effects
 			(font
@@
 	)
 	(symbol
-		(lib_id "power:PWR_FLAG")
-		(at 257.81 29.21 0)
-		(unit 1)
-		(body_style 1)
-		(exclude_from_sim no)
-		(in_bom yes)
-		(on_board yes)
-		(in_pos_files yes)
-		(dnp no)
-		(fields_autoplaced yes)
-		(property "Reference" "#FLG01"
-			(at 257.81 27.305 0)
-			(hide yes)
-			(show_name no)
-			(do_not_autoplace no)
-			(effects
-				(font
-					(size 1.27 1.27)
-				)
-			)
-		)
-		(property "Value" "PWR_FLAG"
-			(at 257.81 24.13 0)
-			(show_name no)
-			(do_not_autoplace no)
-			(effects
-				(font
-					(size 1.27 1.27)
-				)
-			)
-		)
-		(property "Footprint" ""
-			(at 257.81 29.21 0)
-			(hide yes)
-			(show_name no)
-			(do_not_autoplace no)
-			(effects
-				(font
-					(size 1.27 1.27)
-				)
-			)
-		)
-		(property "Datasheet" ""
-			(at 257.81 29.21 0)
-			(hide yes)
-			(show_name no)
-			(do_not_autoplace no)
-			(effects
-				(font
-					(size 1.27 1.27)
-				)
-			)
-		)
-		(property "Description" "Special symbol for telling ERC where power comes from"
-			(at 257.81 29.21 0)
-			(hide yes)
-			(show_name no)
-			(do_not_autoplace no)
-			(effects
-				(font
-					(size 1.27 1.27)
-				)
-			)
-		)
-		(pin "1"
-		)
-		(instances
-			(project "MCU Datalogger"
-				(path "/39677551-78dc-499d-bb11-ebea4292d876"
-					(reference "#FLG01")
-					(unit 1)
-				)
-			)
-		)
-	)
-	(symbol
 		(lib_id "Device:LED")
 		(at 257.81 54.61 90)
@@
 		)
 		(pin "MISO" output
-			(at 151.13 139.7 180)
+			(at 151.13 146.05 180)
 			(effects
 				(font
@@
 		)
 		(pin "MOSI" input
-			(at 151.13 143.51 180)
+			(at 151.13 148.59 180)
 			(effects
 				(font
@@
 		)
 		(pin "RESET" passive
-			(at 151.13 151.13 180)
+			(at 151.13 152.4 180)
 			(effects
 				(font
@@
 			)
 		)
-		(pin "SCK" passive
-			(at 151.13 134.62 180)
+		(pin "SDA" bidirectional
+			(at 151.13 133.35 180)
 			(effects
 				(font
@@
 			)
 		)
-		(pin "SDA" bidirectional
-			(at 151.13 132.08 180)
+		(pin "TX" output
+			(at 151.13 127 180)
 			(effects
 				(font
@@
 			)
 		)
-		(pin "TX" output
-			(at 151.13 127 180)
+		(pin "VCC" passive
+			(at 151.13 119.38 180)
 			(effects
 				(font
@@
 			)
 		)
-		(pin "VCC" passive
-			(at 151.13 119.38 180)
+		(pin "SCK" passive
+			(at 151.13 138.43 180)
+			(effects
+				(font
+					(size 1.27 1.27)
+				)
+				(justify left)
+			)
+		)
+		(pin "SCL" passive
+			(at 151.13 135.89 180)
 			(effects
 				(font
