File: MCU Datalogger.kicad_pcb (KiCad board)
At the start: 2 copper layers, 61 x 40.6 mm, 30 parts, among them J1 Conn_01x04_Pin, J2 Conn_01x04_Pin, J3 Conn_01x09_Pin, J4 Conn_02x03_Odd_Even, U1 24LC1025, U2 24LC1025, U3 DS1337S_, U4 ATMEGA328P-AU, Y1 16MHz, Y2 32.768 KHz

Commit message: First progress on the four layered branch
Parts:
- moved REF** 53.2 mm to (161.6, 63.2)
Routing:
- net GND: track 257.1 -> 0.00 mm
- net /VCC: track 380.0 -> 194.2 mm, vias 11 -> 6
- net /SDA: track 185.1 -> 0.00 mm, vias 8 -> 0
- net /SCK: track 157.5 -> 63.7 mm, vias 3 -> 4
- net Net-(D1-K): track 49.5 -> 0.00 mm, vias 4 -> 0
- net Net-(U4-PB6): track 86.4 -> 38.3 mm, vias 4 -> 0
- net Net-(D2-K): track 45.7 -> 0.00 mm, vias 4 -> 0
- net Net-(U3-SQW/~INT): track 40.2 -> 0.00 mm, vias 4 -> 0
- net /RESET: track 47.9 -> 9.25 mm, vias 3 -> 0
- net Net-(U3-~{INTA}): track 35.0 -> 0.00 mm, vias 2 -> 0
- net /TX: track 65.2 -> 38.7 mm, vias 2 -> 0
- net /RX: track 61.2 -> 36.2 mm, vias 1 -> 0
- net /D4: track 50.9 -> 26.4 mm, vias 1 -> 0
- net /D3: track 49.8 -> 28.9 mm, vias 4 -> 0
- net Net-(U3-X1): track 24.7 -> 44.0 mm, vias 2 -> 0
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Other:
- copper layers 2 -> 4

Commit message: Completed 4 Layered PCB routing
Parts:
- moved REF** 57.5 mm to (104.1, 62.4)
Routing:
- net GND: track 0.00 -> 173.8 mm, vias 0 -> 25
- net /SDA: track 0.00 -> 96.9 mm, vias 0 -> 10
- net Net-(U3-SQW/~INT): track 0.00 -> 45.8 mm, vias 0 -> 2
- net /SCK: track 63.7 -> 101.4 mm, vias 4 -> 11
- net /VCC: track 194.2 -> 226.0 mm, vias 6 -> 10
- net Net-(U3-~{INTA}): track 0.00 -> 29.7 mm, vias 0 -> 2
- net /RESET: track 9.25 -> 35.6 mm, vias 0 -> 2
- net Net-(U4-PB7): track 32.1 -> 56.3 mm, vias 2 -> 4
- net Net-(U4-PB6): track 38.3 -> 48.2 mm, vias 0 -> 2
- net Net-(D2-K): track 0.00 -> 6.80 mm, vias 0 -> 2
- net Net-(D1-K): track 0.00 -> 6.41 mm
- net /D4: track 26.4 -> 28.1 mm
- net Net-(U3-X2): track 36.0 -> 36.9 mm
- net /D5: track 20.1 -> 20.7 mm
